File: Adacel.kicad_pcb (KiCad board)
At the start: 2 copper layers, 65 x 56 mm, 19 parts, among them J1 GPIO, SW1 SW_Push_Dual, SW2 SW_Push_SPDT

Commit message: final gerber files
Parts:
- RV1: footprint Potentiometer_THT:Potentiometer_Piher_PT-10-H01_Horizontal -> Potentiometer_THT:Potentiometer_Piher_PT-10-V05_Vertical
- moved RV1 5.86 mm to (135.5, 75.5)
- moved SW1 3.39 mm to (155.4, 87.3)
- moved R3 2.84 mm to (130.3, 66.8)
- moved D2 2.34 mm to (161.3, 55.4)
- moved C4 2.29 mm to (146.9, 72.6)
- moved U2 1.26 mm to (126.2, 75.0)
- moved C2 0.82 mm to (107.3, 67.1)
Connections:
- J1 pad 1: +3V3 -> +3.3V
Routing:
- net /GPIO22: track 101.6 -> 98.4 mm
- net /GPIO24: track 111.7 -> 109.7 mm
- net Net-(D1-K): track 49.9 -> 51.3 mm
- net Net-(D2-A): track 6.75 -> 5.42 mm
- net +3.3V: track 150.0 -> 149.0 mm
- net Net-(D3-A): track 6.22 -> 5.59 mm
