File: Adacel.kicad_sch (KiCad schematic)
At the start: 15 parts, among them J1 GPIO, SW1 SW_Push_Dual, SW2 SW_Push_SPDT

Commit message: final gerber files
Parts:
- R3: value 500k -> 900k
- RV1: value 1meg -> 220k
Changed lines of the file:
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@@
 	(wire
 		(pts
-			(xy 92.71 24.13) (xy 184.15 24.13)
+			(xy 163.83 46.99) (xy 163.83 36.83)
 		)
 		(stroke
@@
 	(wire
 		(pts
-			(xy 163.83 46.99) (xy 163.83 36.83)
+			(xy 165.1 102.87) (xy 158.75 102.87)
 		)
 		(stroke
@@
 	(wire
 		(pts
-			(xy 165.1 102.87) (xy 158.75 102.87)
-		)
-		(stroke
-			(width 0)
-			(type default)
-		)
-	)
-	(wire
-		(pts
 			(xy 81.28 55.88) (xy 107.95 55.88)
 		)
@@
 			(width 0)
 			(type solid)
-		)
-	)
-	(wire
-		(pts
-			(xy 92.71 15.24) (xy 15.24 15.24)
-		)
-		(stroke
-			(width 0)
-			(type default)
 		)
 	)
@@
 	(wire
 		(pts
-			(xy 15.24 15.24) (xy 15.24 45.72)
+			(xy 180.34 40.64) (xy 181.61 40.64)
 		)
 		(stroke
@@
 	(wire
 		(pts
-			(xy 180.34 40.64) (xy 181.61 40.64)
+			(xy 81.28 76.2) (xy 107.95 76.2)
+		)
+		(stroke
+			(width 0)
+			(type solid)
+		)
+	)
+	(wire
+		(pts
+			(xy 66.04 76.2) (xy 66.04 80.01)
+		)
+		(stroke
+			(width 0)
+			(type solid)
+		)
+	)
+	(wire
+		(pts
+			(xy 63.5 24.13) (xy 63.5 27.94)
+		)
+		(stroke
+			(width 0)
+			(type solid)
+		)
+	)
+	(wire
+		(pts
+			(xy 118.11 106.68) (xy 119.38 106.68)
 		)
 		(stroke
@@
 	(wire
 		(pts
-			(xy 81.28 76.2) (xy 107.95 76.2)
-		)
-		(stroke
-			(width 0)
-			(type solid)
-		)
-	)
-	(wire
-		(pts
-			(xy 66.04 76.2) (xy 66.04 80.01)
-		)
-		(stroke
-			(width 0)
-			(type solid)
-		)
-	)
-	(wire
-		(pts
-			(xy 63.5 24.13) (xy 63.5 27.94)
-		)
-		(stroke
-			(width 0)
-			(type solid)
-		)
-	)
-	(wire
-		(pts
-			(xy 118.11 106.68) (xy 119.38 106.68)
+			(xy 83.82 68.58) (xy 81.28 68.58)
+		)
+		(stroke
+			(width 0)
+			(type solid)
+		)
+	)
+	(wire
+		(pts
+			(xy 39.37 33.02) (xy 68.58 33.02)
+		)
+		(stroke
+			(width 0)
+			(type solid)
+		)
+	)
+	(wire
+		(pts
+			(xy 172.72 30.48) (xy 181.61 30.48)
 		)
 		(stroke
@@
 	(wire
 		(pts
-			(xy 83.82 68.58) (xy 81.28 68.58)
-		)
-		(stroke
-			(width 0)
-			(type solid)
-		)
-	)
-	(wire
-		(pts
-			(xy 39.37 33.02) (xy 68.58 33.02)
-		)
-		(stroke
-			(width 0)
-			(type solid)
-		)
-	)
-	(wire
-		(pts
-			(xy 172.72 30.48) (xy 181.61 30.48)
+			(xy 39.37 55.88) (xy 68.58 55.88)
+		)
+		(stroke
+			(width 0)
+			(type solid)
+		)
+	)
+	(wire
+		(pts
+			(xy 157.48 46.99) (xy 157.48 53.34)
 		)
 		(stroke
@@
 	(wire
 		(pts
-			(xy 39.37 55.88) (xy 68.58 55.88)
-		)
-		(stroke
-			(width 0)
-			(type solid)
-		)
-	)
-	(wire
-		(pts
-			(xy 157.48 46.99) (xy 157.48 53.34)
+			(xy 68.58 30.48) (xy 39.37 30.48)
+		)
+		(stroke
+			(width 0)
+			(type solid)
+		)
+	)
+	(wire
+		(pts
+			(xy 81.28 40.64) (xy 107.95 40.64)
+		)
+		(stroke
+			(width 0)
+			(type solid)
+		)
+	)
+	(wire
+		(pts
+			(xy 83.82 24.13) (xy 83.82 27.94)
+		)
+		(stroke
+			(width 0)
+			(type solid)
+		)
+	)
+	(wire
+		(pts
+			(xy 165.1 107.95) (xy 158.75 107.95)
 		)
 		(stroke
@@
 	(wire
 		(pts
-			(xy 68.58 30.48) (xy 39.37 30.48)
-		)
-		(stroke
-			(width 0)
-			(type solid)
-		)
-	)
-	(wire
-		(pts
-			(xy 15.24 45.72) (xy 68.58 45.72)
+			(xy 39.37 35.56) (xy 68.58 35.56)
+		)
+		(stroke
+			(width 0)
+			(type solid)
+		)
+	)
+	(wire
+		(pts
+			(xy 83.82 27.94) (xy 81.28 27.94)
+		)
+		(stroke
+			(width 0)
+			(type solid)
+		)
+	)
+	(wire
+		(pts
+			(xy 81.28 48.26) (xy 107.95 48.26)
+		)
+		(stroke
+			(width 0)
+			(type solid)
+		)
+	)
+	(wire
+		(pts
+			(xy 81.28 38.1) (xy 107.95 38.1)
+		)
+		(stroke
+			(width 0)
+			(type solid)
+		)
+	)
+	(wire
+		(pts
+			(xy 163.83 30.48) (xy 163.83 36.83)
 		)
 		(stroke
@@
 	(wire
 		(pts
-			(xy 81.28 40.64) (xy 107.95 40.64)
-		)
-		(stroke
-			(width 0)
-			(type solid)
-		)
-	)
-	(wire
-		(pts
-			(xy 83.82 24.13) (xy 83.82 27.94)
-		)
-		(stroke
-			(width 0)
-			(type solid)
-		)
-	)
-	(wire
-		(pts
-			(xy 165.1 107.95) (xy 158.75 107.95)
+			(xy 163.83 30.48) (xy 167.64 30.48)
 		)
 		(stroke
@@
 	(wire
 		(pts
-			(xy 39.37 35.56) (xy 68.58 35.56)
-		)
-		(stroke
-			(width 0)
-			(type solid)
-		)
-	)
-	(wire
-		(pts
-			(xy 83.82 27.94) (xy 81.28 27.94)
-		)
-		(stroke
-			(width 0)
-			(type solid)
-		)
-	)
-	(wire
-		(pts
-			(xy 81.28 48.26) (xy 107.95 48.26)
-		)
-		(stroke
-			(width 0)
-			(type solid)
-		)
-	)
-	(wire
-		(pts
-			(xy 81.28 38.1) (xy 107.95 38.1)
-		)
-		(stroke
-			(width 0)
-			(type solid)
-		)
-	)
-	(wire
-		(pts
-			(xy 92.71 24.13) (xy 92.71 15.24)
-		)
-		(stroke
-			(width 0)
-			(type default)
-		)
-	)
-	(wire
-		(pts
-			(xy 163.83 30.48) (xy 163.83 36.83)
-		)
-		(stroke
-			(width 0)
-			(type default)
-		)
-	)
-	(wire
-		(pts
-			(xy 163.83 30.48) (xy 167.64 30.48)
-		)
-		(stroke
-			(width 0)
-			(type default)
-		)
-	)
-	(wire
-		(pts
 			(xy 39.37 53.34) (xy 68.58 53.34)
 		)
@@
 			(width 0)
 			(type solid)
-		)
-	)
-	(wire
-		(pts
-			(xy 184.15 50.8) (xy 184.15 24.13)
-		)
-		(stroke
-			(width 0)
-			(type default)
 		)
 	)
@@
 	(wire
 		(pts
+			(xy 39.37 45.72) (xy 68.58 45.72)
+		)
+		(stroke
+			(width 0)
+			(type default)
+		)
+	)
+	(wire
+		(pts
 			(xy 68.58 50.8) (xy 39.37 50.8)
 		)
@@
 	(label "GPIO6"
 		(at 39.37 66.04 0)
+		(effects
+			(font
+				(size 1.27 1.27)
+			)
+			(justify left bottom)
+		)
+	)
+	(label "GPIO22"
+		(at 184.15 50.8 0)
 		(effects
 			(font
@@
 			)
 		)
-		(property "Value" "500k"
+		(property "Value" "900k"
 			(at 164.592 39.116 90)
 			(effects
@@
 			)
 		)
-		(property "Value" "1meg"
+		(property "Value" "220k"
 			(at 174.244 42.672 90)
 			(effects
